File: Zprobe Adaptor.sch (KiCad schematic (older format))
At the start: 7 parts, among them J1 Screw_Terminal_01x02, J2 Screw_Terminal_01x02, J3 Screw_Terminal_01x03, U1 LTV-817

Commit message: Updated Parts for Digi-Key
Parts:
- D1: value LED_Small_ALT -> LED; Manufacturer Vishay Semiconductor Opto Division -> Kingbright; Manufacturer Number TLHR4400-MS12Z -> WP937GGD; Supplier Link https://www.digikey.com/products/en?keywords=TLHR4400-MS12Z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 -> https://www.digikey.com/products/en?keywords=754-2199-ND; Supplier Part No TLHR4400-MS12ZTB-ND -> 754-2199-ND
Changed lines of the file:
@@
 P 5125 3975
 F 0 "D1" V 5125 3907 50  0000 R CNN
-F 1 "LED_Small_ALT" V 5080 3907 50  0001 R CNN
+F 1 "LED" V 5080 3907 50  0001 R CNN
 F 2 "LEDs:LED_D3.0mm" V 5125 3975 50  0001 C CNN
-F 3 "http://www.vishay.com/docs/83006/tlhg440.pdf" V 5125 3975 50  0001 C CNN
-F 4 "TLHR4400-MS12Z" H 5125 3975 50  0001 C CNN "Manufacturer Number"
+F 3 "http://www.kingbrightusa.com/images/catalog/SPEC/WP937GGD.pdf" V 5125 3975 50  0001 C CNN
+F 4 "WP937GGD" H 5125 3975 50  0001 C CNN "Manufacturer Number"
 F 5 "Digi-Key" H 5125 3975 50  0001 C CNN "Supplier"
-F 6 "TLHR4400-MS12ZTB-ND" H 5125 3975 50  0001 C CNN "Supplier Part No"
-F 7 "https://www.digikey.com/products/en?keywords=TLHR4400-MS12ZTB-ND" H 5125 3975 50  0001 C CNN "Supplier Link"
-F 8 "Vishay Semiconductor Opto Division" H 5125 3975 50  0001 C CNN "Manufacturer"
+F 6 "754-2199-ND" H 5125 3975 50  0001 C CNN "Supplier Part No"
+F 7 "https://www.digikey.com/products/en?keywords=754-2199-ND" H 5125 3975 50  0001 C CNN "Supplier Link"
+F 8 "Kingbright" H 5125 3975 50  0001 C CNN "Manufacturer"
 	1    5125 3975
 	0    -1   -1   0
